Commit message: TF set perfect, static broadcaster.

File: carla_ad_demo/launch/tesla.urdf (robot description, URDF)
Before this commit: robot mbot, 3 links, 2 joints
Links:
- removed link left_wheel_link
- removed link right_wheel_link
Joints:
- removed joint left_wheel_joint
- removed joint right_wheel_joint
